File: PCB/MagStrike.kicad_sch (KiCad schematic)
At the start: 0 parts

Commit message: added lots of kicad stuff
Parts:
- added A1: RaspberryPi_Pico, Module:RaspberryPi_Pico_Common_Unspecified, symbol MCU_Module:RaspberryPi_Pico
- added SW1, SW10, SW11, SW12, SW13, SW14, SW15, SW16, SW17, SW18, SW19, SW2, SW20, SW21, SW22, SW23, SW24, SW25, SW26, SW27, SW28, SW29, SW3, SW30, SW31, SW32, SW33, SW34, SW35, SW36, SW37, SW38, SW39, SW4, SW40, SW41, SW42, SW43, SW44, SW45, SW46, SW47, SW48, SW49, SW5, SW50, SW51, SW52, SW53, SW54, SW55, SW56, SW57, SW58, SW59, SW6, SW60, SW61, SW7, SW8, SW9: ~, symbol MagStrike:HESW
- added U1, U2, U3, U4: CD74HC4067M96, digikey-footprints:SOIC-24_W7.50mm, symbol dk_Interface-Analog-Switches-Multiplexers-Demultiplexers:CD74HC4067M96
Connections:
- new net: SW41.1 (VCC), SW41.4 (C1)
- new net: SW41.2 (GND), SW41.5 (C2)
- new net: SW44.1 (VCC), SW44.4 (C1)
- new net: SW44.2 (GND), SW44.5 (C2)
- new net: SW42.1 (VCC), SW42.4 (C1)
- new net: SW42.2 (GND), SW42.5 (C2)
- new net: SW16.1 (VCC), SW16.4 (C1)
- new net: SW16.2 (GND), SW16.5 (C2)
- new net: SW46.1 (VCC), SW46.4 (C1)
- new net: SW46.2 (GND), SW46.5 (C2)
- new net: SW50.1 (VCC), SW50.4 (C1)
- new net: SW50.2 (GND), SW50.5 (C2)
- new net: SW19.1 (VCC), SW19.4 (C1)
- new net: SW19.2 (GND), SW19.5 (C2)
- new net: SW20.1 (VCC), SW20.4 (C1)
- new net: SW20.2 (GND), SW20.5 (C2)
- new net: SW10.1 (VCC), SW10.4 (C1)
- new net: SW10.2 (GND), SW10.5 (C2)
- new net: SW22.1 (VCC), SW22.4 (C1)
- new net: SW22.2 (GND), SW22.5 (C2)
- new net: SW34.1 (VCC), SW34.4 (C1)
- new net: SW34.2 (GND), SW34.5 (C2)
- new net: SW55.1 (VCC), SW55.4 (C1)
- new net: SW55.2 (GND), SW55.5 (C2)
- new net: SW33.1 (VCC), SW33.4 (C1)
- new net: SW33.2 (GND), SW33.5 (C2)
- new net: SW15.1 (VCC), SW15.4 (C1)
- new net: SW15.2 (GND), SW15.5 (C2)
- new net: SW3.1 (VCC), SW3.4 (C1)
- new net: SW3.2 (GND), SW3.5 (C2)
- new net: SW7.1 (VCC), SW7.4 (C1)
- new net: SW7.2 (GND), SW7.5 (C2)
- new net: SW25.1 (VCC), SW25.4 (C1)
- new net: SW25.2 (GND), SW25.5 (C2)
- new net: SW2.1 (VCC), SW2.4 (C1)
- new net: SW2.2 (GND), SW2.5 (C2)
- new net: SW56.1 (VCC), SW56.4 (C1)
- new net: SW56.2 (GND), SW56.5 (C2)
- new net: SW51.1 (VCC), SW51.4 (C1)
- new net: SW51.2 (GND), SW51.5 (C2)
- new net: SW27.1 (VCC), SW27.4 (C1)
- new net: SW27.2 (GND), SW27.5 (C2)
- new net: SW40.1 (VCC), SW40.4 (C1)
- new net: SW40.2 (GND), SW40.5 (C2)
- new net: SW8.1 (VCC), SW8.4 (C1)
- new net: SW8.2 (GND), SW8.5 (C2)
- new net: SW1.1 (VCC), SW1.4 (C1)
- new net: SW1.2 (GND), SW1.5 (C2)
- new net: SW59.1 (VCC), SW59.4 (C1)
- new net: SW59.2 (GND), SW59.5 (C2)
- new net: SW61.1 (VCC), SW61.4 (C1)
- new net: SW61.2 (GND), SW61.5 (C2)
- new net: SW38.1 (VCC), SW38.4 (C1)
- new net: SW38.2 (GND), SW38.5 (C2)
- new net: SW5.1 (VCC), SW5.4 (C1)
- new net: SW5.2 (GND), SW5.5 (C2)
- new net: SW24.1 (VCC), SW24.4 (C1)
- new net: SW24.2 (GND), SW24.5 (C2)
- new net: SW23.1 (VCC), SW23.4 (C1)
- new net: SW23.2 (GND), SW23.5 (C2)
- new net: SW17.1 (VCC), SW17.4 (C1)
- new net: SW17.2 (GND), SW17.5 (C2)
- new net: SW48.1 (VCC), SW48.4 (C1)
- new net: SW48.2 (GND), SW48.5 (C2)
- new net: SW29.1 (VCC), SW29.4 (C1)
- new net: SW29.2 (GND), SW29.5 (C2)
- new net: SW6.1 (VCC), SW6.4 (C1)
- new net: SW6.2 (GND), SW6.5 (C2)
- new net: SW43.1 (VCC), SW43.4 (C1)
- new net: SW43.2 (GND), SW43.5 (C2)
- new net: SW58.1 (VCC), SW58.4 (C1)
- new net: SW58.2 (GND), SW58.5 (C2)
- new net: SW45.1 (VCC), SW45.4 (C1)
- new net: SW45.2 (GND), SW45.5 (C2)
- new net: SW26.1 (VCC), SW26.4 (C1)
- new net: SW26.2 (GND), SW26.5 (C2)
- new net: SW53.1 (VCC), SW53.4 (C1)
- new net: SW53.2 (GND), SW53.5 (C2)
- new net: SW18.1 (VCC), SW18.4 (C1)
- new net: SW18.2 (GND), SW18.5 (C2)
- new net: SW9.1 (VCC), SW9.4 (C1)
- new net: SW9.2 (GND), SW9.5 (C2)
- new net: SW31.1 (VCC), SW31.4 (C1)
- new net: SW31.2 (GND), SW31.5 (C2)
- new net: SW39.1 (VCC), SW39.4 (C1)
- new net: SW39.2 (GND), SW39.5 (C2)
- new net: SW54.1 (VCC), SW54.4 (C1)
- new net: SW54.2 (GND), SW54.5 (C2)
- new net: SW52.1 (VCC), SW52.4 (C1)
- new net: SW52.2 (GND), SW52.5 (C2)
- new net: SW13.1 (VCC), SW13.4 (C1)
- new net: SW13.2 (GND), SW13.5 (C2)
- new net: SW36.1 (VCC), SW36.4 (C1)
- new net: SW36.2 (GND), SW36.5 (C2)
- new net: SW11.1 (VCC), SW11.4 (C1)
- new net: SW11.2 (GND), SW11.5 (C2)
- new net: SW21.1 (VCC), SW21.4 (C1)
- new net: SW21.2 (GND), SW21.5 (C2)
- new net: SW28.1 (VCC), SW28.4 (C1)
- new net: SW28.2 (GND), SW28.5 (C2)
- new net: A1.13 (GND), A1.18 (GND), A1.23 (GND), A1.28 (GND), A1.3 (GND), A1.38 (GND), A1.8 (GND)
- new net: SW30.1 (VCC), SW30.4 (C1)
- new net: SW30.2 (GND), SW30.5 (C2)
- new net: SW47.1 (VCC), SW47.4 (C1)
- new net: SW47.2 (GND), SW47.5 (C2)
- new net: SW49.1 (VCC), SW49.4 (C1)
- new net: SW49.2 (GND), SW49.5 (C2)
- new net: SW32.1 (VCC), SW32.4 (C1)
- new net: SW32.2 (GND), SW32.5 (C2)
- new net: SW60.1 (VCC), SW60.4 (C1)
- new net: SW60.2 (GND), SW60.5 (C2)
- new net: SW37.1 (VCC), SW37.4 (C1)
- new net: SW37.2 (GND), SW37.5 (C2)
- new net: SW57.1 (VCC), SW57.4 (C1)
- new net: SW57.2 (GND), SW57.5 (C2)
- new net: SW14.1 (VCC), SW14.4 (C1)
- new net: SW14.2 (GND), SW14.5 (C2)
- new net: SW12.1 (VCC), SW12.4 (C1)
- new net: SW12.2 (GND), SW12.5 (C2)
- new net: SW35.1 (VCC), SW35.4 (C1)
- new net: SW35.2 (GND), SW35.5 (C2)
- new net: SW4.1 (VCC), SW4.4 (C1)
- new net: SW4.2 (GND), SW4.5 (C2)
- new net GPIO0: A1.1 (GPIO0)

Commit message: added stuff
Parts:
- removed U1, U2, U3, U4: CD74HC4067M96, digikey-footprints:SOIC-24_W7.50mm, symbol dk_Interface-Analog-Switches-Multiplexers-Demultiplexers:CD74HC4067M96
- added U1, U2, U3, U4: CD74HC4067M, Package_SO:SOIC-24W_7.5x15.4mm_P1.27mm, symbol 74xx:CD74HC4067M
Connections:
- net +3V3: now reaches SW41.1 (VCC), SW41.4 (C1)
- net +3V3: now also A1.36 (3V3), SW1.1 (VCC), SW1.4 (C1), SW10.1 (VCC), SW10.4 (C1), SW11.1 (VCC), SW11.4 (C1), SW12.1 (VCC), SW12.4 (C1), SW13.1 (VCC), SW13.4 (C1), SW14.1 (VCC), SW14.4 (C1), SW15.1 (VCC), SW15.4 (C1), SW16.1 (VCC), SW16.4 (C1), SW17.1 (VCC), SW17.4 (C1), SW18.1 (VCC), SW18.4 (C1), SW19.1 (VCC), SW19.4 (C1), SW2.1 (VCC), SW2.4 (C1), SW20.1 (VCC), SW20.4 (C1), SW21.1 (VCC), SW21.4 (C1), SW22.1 (VCC), SW22.4 (C1), SW23.1 (VCC), SW23.4 (C1), SW24.1 (VCC), SW24.4 (C1), SW25.1 (VCC), SW25.4 (C1), SW26.1 (VCC), SW26.4 (C1), SW27.1 (VCC), SW27.4 (C1), SW28.1 (VCC), SW28.4 (C1), SW29.1 (VCC), SW29.4 (C1), SW3.1 (VCC), SW3.4 (C1), SW30.1 (VCC), SW30.4 (C1), SW31.1 (VCC), SW31.4 (C1), SW32.1 (VCC), SW32.4 (C1), SW33.1 (VCC), SW33.4 (C1), SW34.1 (VCC), SW34.4 (C1), SW35.1 (VCC), SW35.4 (C1), SW36.1 (VCC), SW36.4 (C1), SW37.1 (VCC), SW37.4 (C1), SW38.1 (VCC), SW38.4 (C1), SW39.1 (VCC), SW39.4 (C1), SW4.1 (VCC), SW4.4 (C1), SW40.1 (VCC), SW40.4 (C1), SW42.1 (VCC), SW42.4 (C1), SW43.1 (VCC), SW43.4 (C1), SW44.1 (VCC), SW44.4 (C1), SW45.1 (VCC), SW45.4 (C1), SW46.1 (VCC), SW46.4 (C1), SW47.1 (VCC), SW47.4 (C1), SW48.1 (VCC), SW48.4 (C1), SW49.1 (VCC), SW49.4 (C1), SW5.1 (VCC), SW5.4 (C1), SW50.1 (VCC), SW50.4 (C1), SW51.1 (VCC), SW51.4 (C1), SW52.1 (VCC), SW52.4 (C1), SW53.1 (VCC), SW53.4 (C1), SW54.1 (VCC), SW54.4 (C1), SW55.1 (VCC), SW55.4 (C1), SW56.1 (VCC), SW56.4 (C1), SW57.1 (VCC), SW57.4 (C1), SW58.1 (VCC), SW58.4 (C1), SW59.1 (VCC), SW59.4 (C1), SW6.1 (VCC), SW6.4 (C1), SW60.1 (VCC), SW60.4 (C1), SW61.1 (VCC), SW61.4 (C1), SW7.1 (VCC), SW7.4 (C1), SW8.1 (VCC), SW8.4 (C1), SW9.1 (VCC), SW9.4 (C1), U1.24 (VCC), U2.24 (VCC), U3.24 (VCC), U4.24 (VCC)
- net GND: now reaches SW41.2 (GND), SW41.5 (C2)
- net GND: now also A1.13 (GND), A1.18 (GND), A1.23 (GND), A1.28 (GND), A1.3 (GND), A1.38 (GND), A1.8 (GND), SW1.2 (GND), SW1.5 (C2), SW10.2 (GND), SW10.5 (C2), SW11.2 (GND), SW11.5 (C2), SW12.2 (GND), SW12.5 (C2), SW13.2 (GND), SW13.5 (C2), SW14.2 (GND), SW14.5 (C2), SW15.2 (GND), SW15.5 (C2), SW16.2 (GND), SW16.5 (C2), SW17.2 (GND), SW17.5 (C2), SW18.2 (GND), SW18.5 (C2), SW19.2 (GND), SW19.5 (C2), SW2.2 (GND), SW2.5 (C2), SW20.2 (GND), SW20.5 (C2), SW21.2 (GND), SW21.5 (C2), SW22.2 (GND), SW22.5 (C2), SW23.2 (GND), SW23.5 (C2), SW24.2 (GND), SW24.5 (C2), SW25.2 (GND), SW25.5 (C2), SW26.2 (GND), SW26.5 (C2), SW27.2 (GND), SW27.5 (C2), SW28.2 (GND), SW28.5 (C2), SW29.2 (GND), SW29.5 (C2), SW3.2 (GND), SW3.5 (C2), SW30.2 (GND), SW30.5 (C2), SW31.2 (GND), SW31.5 (C2), SW32.2 (GND), SW32.5 (C2), SW33.2 (GND), SW33.5 (C2), SW34.2 (GND), SW34.5 (C2), SW35.2 (GND), SW35.5 (C2), SW36.2 (GND), SW36.5 (C2), SW37.2 (GND), SW37.5 (C2), SW38.2 (GND), SW38.5 (C2), SW39.2 (GND), SW39.5 (C2), SW4.2 (GND), SW4.5 (C2), SW40.2 (GND), SW40.5 (C2), SW42.2 (GND), SW42.5 (C2), SW43.2 (GND), SW43.5 (C2), SW44.2 (GND), SW44.5 (C2), SW45.2 (GND), SW45.5 (C2), SW46.2 (GND), SW46.5 (C2), SW47.2 (GND), SW47.5 (C2), SW48.2 (GND), SW48.5 (C2), SW49.2 (GND), SW49.5 (C2), SW5.2 (GND), SW5.5 (C2), SW50.2 (GND), SW50.5 (C2), SW51.2 (GND), SW51.5 (C2), SW52.2 (GND), SW52.5 (C2), SW53.2 (GND), SW53.5 (C2), SW54.2 (GND), SW54.5 (C2), SW55.2 (GND), SW55.5 (C2), SW56.2 (GND), SW56.5 (C2), SW57.2 (GND), SW57.5 (C2), SW58.2 (GND), SW58.5 (C2), SW59.2 (GND), SW59.5 (C2), SW6.2 (GND), SW6.5 (C2), SW60.2 (GND), SW60.5 (C2), SW61.2 (GND), SW61.5 (C2), SW7.2 (GND), SW7.5 (C2), SW8.2 (GND), SW8.5 (C2), SW9.2 (GND), SW9.5 (C2), U1.12 (GND), U2.12 (GND), U3.12 (GND), U4.12 (GND)
- net SW41: now reaches SW41.3 (OUT)
- net SW41: now also U3.23 (I8)
- net SW44: now reaches SW44.3 (OUT)
- net SW44: now also U3.20 (I11)
- net SW42: now reaches SW42.3 (OUT)
- net SW42: now also U3.22 (I9)
- net SW16: now reaches SW16.3 (OUT)
- net SW16: now also U1.16 (I15)
- net SW46: now reaches SW46.3 (OUT)
- net SW46: now also U3.18 (I13)
- net SW50: now reaches SW50.3 (OUT)
- net SW50: now also U4.8 (I1)
- net SW19: now reaches SW19.3 (OUT)
- net SW19: now also U2.7 (I2)
- net SW20: now reaches SW20.3 (OUT)
- net SW20: now also U2.6 (I3)
- net SW10: now reaches SW10.3 (OUT)
- net SW10: now also U1.22 (I9)
- net SW22: now reaches SW22.3 (OUT)
- net SW22: now also U2.4 (I5)
- net SW34: now reaches SW34.3 (OUT)
- net SW34: now also U3.8 (I1)
- net SW55: now reaches SW55.3 (OUT)
- net SW55: now also U4.3 (I6)
- net SW33: now reaches SW33.3 (OUT)
- net SW33: now also U3.9 (I0)
- net SW15: now reaches SW15.3 (OUT)
- net SW15: now also U1.17 (I14)
- net SW3: now reaches SW3.3 (OUT)
- net SW3: now also U1.7 (I2)
- net SW7: now reaches SW7.3 (OUT)
- net SW7: now also U1.3 (I6)
- net SW25: now reaches SW25.3 (OUT)
- net SW25: now also U2.23 (I8)
- net SW2: now reaches SW2.3 (OUT)
- net SW2: now also U1.8 (I1)
- net SW56: now reaches SW56.3 (OUT)
- net SW56: now also U4.2 (I7)
- net SW51: now reaches SW51.3 (OUT)
- net SW51: now also U4.7 (I2)
- net SW27: now reaches SW27.3 (OUT)
- net SW27: now also U2.21 (I10)
- net SW40: now reaches SW40.3 (OUT)
- net SW40: now also U3.2 (I7)
- net SW8: now reaches SW8.3 (OUT)
- net SW8: now also U1.2 (I7)
- net SW1: now reaches SW1.3 (OUT)
- net SW1: now also U1.9 (I0)
- net SW59: now reaches SW59.3 (OUT)
- net SW59: now also U4.21 (I10)
- net SW61: now reaches SW61.3 (OUT)
- net SW61: now also U4.19 (I12)
- net SW38: now reaches SW38.3 (OUT)
- net SW38: now also U3.4 (I5)
- net SW5: now reaches SW5.3 (OUT)
- net SW5: now also U1.5 (I4)
- net SW24: now reaches SW24.3 (OUT)
- net SW24: now also U2.2 (I7)
- net SW23: now reaches SW23.3 (OUT)
- net SW23: now also U2.3 (I6)
- net SW17: now reaches SW17.3 (OUT)
- net SW17: now also U2.9 (I0)
- net SW48: now reaches SW48.3 (OUT)
- net SW48: now also U3.16 (I15)
- net SW29: now reaches SW29.3 (OUT)
- net SW29: now also U2.19 (I12)
- net SW6: now reaches SW6.3 (OUT)
- net SW6: now also U1.4 (I5)
- net SW43: now reaches SW43.3 (OUT)
- net SW43: now also U3.21 (I10)
- net SW58: now reaches SW58.3 (OUT)
- net SW58: now also U4.22 (I9)
- net SW45: now reaches SW45.3 (OUT)
- net SW45: now also U3.19 (I12)
- net SW26: now reaches SW26.3 (OUT)
- net SW26: now also U2.22 (I9)
- net SW53: now reaches SW53.3 (OUT)
- net SW53: now also U4.5 (I4)
- net SW18: now reaches SW18.3 (OUT)
- net SW18: now also U2.8 (I1)
- net SW9: now reaches SW9.3 (OUT)
- net SW9: now also U1.23 (I8)
- net SW31: now reaches SW31.3 (OUT)
- net SW31: now also U2.17 (I14)
- net SW39: now reaches SW39.3 (OUT)
- net SW39: now also U3.3 (I6)
- net SW54: now reaches SW54.3 (OUT)
- net SW54: now also U4.4 (I5)
- net SW52: now reaches SW52.3 (OUT)
- net SW52: now also U4.6 (I3)
- net SW13: now reaches SW13.3 (OUT)
- net SW13: now also U1.19 (I12)
- net SW36: now reaches SW36.3 (OUT)
- net SW36: now also U3.6 (I3)
- net SW11: now reaches SW11.3 (OUT)
- net SW11: now also U1.21 (I10)
- net SW21: now reaches SW21.3 (OUT)
- net SW21: now also U2.5 (I4)
- net SW28: now reaches SW28.3 (OUT)
- net SW28: now also U2.20 (I11)
- net GPI07: now reaches A1.10 (GPIO7)
- net GPI08: now reaches A1.11 (GPIO8)
- net GPI08: now also U1.10 (S0), U2.10 (S0), U3.10 (S0), U4.10 (S0)
- net GPI09: now reaches A1.12 (GPIO9)
- net GPI09: now also U1.11 (S1), U2.11 (S1), U3.11 (S1), U4.11 (S1)
- net GPI010: now reaches A1.14 (GPIO10)
- net GPI010: now also U1.14 (S2), U2.14 (S2), U3.14 (S2), U4.14 (S2)
- net GPI011: now reaches A1.15 (GPIO11)
- net GPI011: now also U1.13 (S3), U2.13 (S3), U3.13 (S3), U4.13 (S3)
- net GPI012: now reaches A1.16 (GPIO12)
- net GPI012: now also U1.15 (~{E})
- net GPI013: now reaches A1.17 (GPIO13)
- net GPI013: now also U2.15 (~{E})
- net GPI014: now reaches A1.19 (GPIO14)
- net GPI014: now also U3.15 (~{E})
- net GPIO1: now reaches A1.2 (GPIO1)
- net GPIO15: now reaches A1.20 (GPIO15)
- net GPI016: now reaches A1.21 (GPIO16)
- net GPI017: now reaches A1.22 (GPIO17)
- net GPI018: now reaches A1.24 (GPIO18)
- net GPI019: now reaches A1.25 (GPIO19)
- net GPI020: now reaches A1.26 (GPIO20)
- net GPI021: now reaches A1.27 (GPIO21)
- net GPI022: now reaches A1.29 (GPIO22)
- net GPI026_ADC0: now reaches A1.31 (GPIO26_ADC0)
- net GPI027_ADC1: now reaches A1.32 (GPIO27_ADC1)
- net GPI028_ADC2: now reaches A1.34 (GPIO28_ADC2)
- net ADC_VREF: now reaches A1.35 (ADC_VREF)
- net GPIO2: now reaches A1.4 (GPIO2)
- net GPIO3: now reaches A1.5 (GPIO3)
- net GPIO4: now reaches A1.6 (GPIO4)
- net GPI05: now reaches A1.7 (GPIO5)
- net GPI06: now reaches A1.9 (GPIO6)
- net SW30: now reaches SW30.3 (OUT)
- net SW30: now also U2.18 (I13)
- net SW47: now reaches SW47.3 (OUT)
- net SW47: now also U3.17 (I14)
- net SW49: now reaches SW49.3 (OUT)
- net SW49: now also U4.9 (I0)
- net SW32: now reaches SW32.3 (OUT)
- net SW32: now also U2.16 (I15)
- net SW60: now reaches SW60.3 (OUT)
- net SW60: now also U4.20 (I11)
- net SW37: now reaches SW37.3 (OUT)
- net SW37: now also U3.5 (I4)
- net SW57: now reaches SW57.3 (OUT)
- net SW57: now also U4.23 (I8)
- net SW14: now reaches SW14.3 (OUT)
- net SW14: now also U1.18 (I13)
- net SW12: now reaches SW12.3 (OUT)
- net SW12: now also U1.20 (I11)
- net SW35: now reaches SW35.3 (OUT)
- net SW35: now also U3.7 (I2)
- net SW4: now reaches SW4.3 (OUT)
- net SW4: now also U1.6 (I3)
- new net GPI015: U4.15 (~{E})
- new net GPI026: U1.1 (COM), U2.1 (COM), U3.1 (COM), U4.1 (COM)
