File: PCB/MagStrike.kicad_sch (KiCad schematic)
At the start: 66 parts, among them U1 CD74HC4067M, U2 CD74HC4067M, U3 CD74HC4067M, U4 CD74HC4067M

Commit message: s
Connections:
- net ADC_VREF is gone; now on net +3V3: A1.35 (ADC_VREF)
- net GPI015 is gone; now on net GPIO15: U4.15 (~{E})
- no-connect marks 0 -> 8
Changed lines of the file:
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@@
 		(color 0 0 0 0)
 	)
+	(no_connect
+		(at 273.05 92.71)
+	)
+	(no_connect
+		(at 381 171.45)
+	)
+	(no_connect
+		(at 227.33 49.53)
+	)
+	(no_connect
+		(at 250.19 31.75)
+	)
+	(no_connect
+		(at 381 168.91)
+	)
+	(no_connect
+		(at 381 173.99)
+	)
+	(no_connect
+		(at 227.33 46.99)
+	)
+	(no_connect
+		(at 245.11 31.75)
+	)
 	(wire
 		(pts
@@
 	(wire
 		(pts
+			(xy 354.33 168.91) (xy 355.6 168.91)
+		)
+		(stroke
+			(width 0)
+			(type default)
+		)
+	)
+	(wire
+		(pts
 			(xy 59.69 86.36) (xy 50.8 86.36)
 		)
@@
 	(wire
 		(pts
+			(xy 226.06 92.71) (xy 227.33 92.71)
+		)
+		(stroke
+			(width 0)
+			(type default)
+		)
+	)
+	(wire
+		(pts
 			(xy 59.69 234.95) (xy 55.88 234.95)
 		)
@@
 	(global_label "GPIO15"
 		(shape input)
-		(at 227.33 92.71 180)
+		(at 226.06 92.71 180)
 		(fields_autoplaced yes)
 		(effects
@@
 		)
 		(property "Intersheetrefs" "${INTERSHEET_REFS}"
-			(at 217.4505 92.71 0)
+			(at 216.1805 92.71 0)
 			(effects
 				(font
@@
 		)
 	)
-	(global_label "GPI015"
+	(global_label "GPIO15"
 		(shape input)
-		(at 355.6 168.91 180)
+		(at 354.33 168.91 180)
 		(fields_autoplaced yes)
 		(effects
@@
 		)
 		(property "Intersheetrefs" "${INTERSHEET_REFS}"
-			(at 345.8415 168.91 0)
+			(at 344.4505 168.91 0)
 			(effects
 				(font
@@
 		)
 	)
-	(global_label "ADC_VREF"
-		(shape input)
-		(at 273.05 77.47 0)
-		(fields_autoplaced yes)
-		(effects
-			(font
-				(size 1.27 1.27)
-			)
-			(justify left)
-		)
-		(property "Intersheetrefs" "${INTERSHEET_REFS}"
-			(at 285.2276 77.47 0)
-			(effects
-				(font
-					(size 1.27 1.27)
-				)
-				(justify left)
-				(hide yes)
-			)
-		)
-	)
 	(global_label "GPI026"
 		(shape input)
@@
 					(unit 1)
 				)
+			)
+		)
+	)
+	(symbol
+		(lib_id "power:+3V3")
+		(at 273.05 77.47 270)
+		(unit 1)
+		(exclude_from_sim no)
+		(in_bom yes)
+		(on_board yes)
+		(dnp no)
+		(fields_autoplaced yes)
+		(property "Reference" "#PWR0133"
+			(at 269.24 77.47 0)
+			(effects
+				(font
+					(size 1.27 1.27)
+				)
+				(hide yes)
+			)
+		)
+		(property "Value" "+3V3"
+			(at 276.86 77.4699 90)
+			(effects
+				(font
+					(size 1.27 1.27)
+				)
+				(justify left)
+			)
+		)
+		(property "Footprint" ""
+			(at 273.05 77.47 0)
+			(effects
+				(font
+					(size 1.27 1.27)
+				)
+				(hide yes)
+			)
+		)
+		(property "Datasheet" ""
+			(at 273.05 77.47 0)
+			(effects
+				(font
+					(size 1.27 1.27)
+				)
+				(hide yes)
+			)
+		)
+		(property "Description" "Power symbol creates a global label with name \"+3V3\""
+			(at 273.05 77.47 0)
+			(effects
+				(font
+					(size 1.27 1.27)
+				)
+				(hide yes)
+			)
+		)
+		(pin "1"
+		)
+		(instances
+			(project "MagStrike"
+				(path "/dbf0735b-e154-44fd-af25-3740650fde67"
+					(reference "#PWR0133")
+					(unit 1)
+				)

Commit message: more stuff
Parts:
- SW1, SW10, SW11, SW12, SW13, SW14, SW15, SW16, SW17, SW18, SW19, SW2, SW20, SW21, SW22, SW23, SW24, SW25, SW26, SW27, SW28, SW29, SW3, SW30, SW31, SW32, SW33, SW34, SW35, SW36, SW37, SW38, SW39, SW4, SW40, SW41, SW42, SW43, SW44, SW45, SW46, SW47, SW48, SW49, SW5, SW50, SW51, SW52, SW53, SW54, SW55, SW56, SW57, SW58, SW59, SW6, SW60, SW61, SW7, SW8, SW9: footprint (none) -> MagStrike:Gateron_Low_Profile_Magnetic_Jade
Changed lines of the file:
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@@
 			)
 		)
-		(property "Footprint" ""
+		(property "Footprint" "MagStrike:Gateron_Low_Profile_Magnetic_Jade"
 			(at 63.5 60.96 0)
 			(effects
@@
 			)
 		)
-		(property "Footprint" ""
+		(property "Footprint" "MagStrike:Gateron_Low_Profile_Magnetic_Jade"
 			(at 33.02 138.43 0)
 			(effects
@@
 			)
 		)
-		(property "Footprint" ""
+		(property "Footprint" "MagStrike:Gateron_Low_Profile_Magnetic_Jade"
 			(at 63.5 162.56 0)
 			(effects
@@
 			)
 		)
-		(property "Footprint" ""
+		(property "Footprint" "MagStrike:Gateron_Low_Profile_Magnetic_Jade"
 			(at 153.67 262.89 0)
 			(effects
@@
 			)
 		)
-		(property "Footprint" ""
+		(property "Footprint" "MagStrike:Gateron_Low_Profile_Magnetic_Jade"
 			(at 63.5 138.43 0)
 			(effects
@@
 			)
 		)
-		(property "Footprint" ""
+		(property "Footprint" "MagStrike:Gateron_Low_Profile_Magnetic_Jade"
 			(at 33.02 262.89 0)
 			(effects
@@
 			)
 		)
-		(property "Footprint" ""
+		(property "Footprint" "MagStrike:Gateron_Low_Profile_Magnetic_Jade"
 			(at 63.5 262.89 0)
 			(effects
@@
 			)
 		)
-		(property "Footprint" ""
+		(property "Footprint" "MagStrike:Gateron_Low_Profile_Magnetic_Jade"
 			(at 33.02 290.83 0)
 			(effects
@@
 			)
 		)
-		(property "Footprint" ""
+		(property "Footprint" "MagStrike:Gateron_Low_Profile_Magnetic_Jade"
 			(at 33.02 162.56 0)
 			(effects
@@
 			)
 		)
-		(property "Footprint" ""
+		(property "Footprint" "MagStrike:Gateron_Low_Profile_Magnetic_Jade"
 			(at 63.5 318.77 0)
 			(effects
@@
 			)
 		)
-		(property "Footprint" ""
+		(property "Footprint" "MagStrike:Gateron_Low_Profile_Magnetic_Jade"
 			(at 124.46 60.96 0)
 			(effects
@@
 			)
 		)
-		(property "Footprint" ""
+		(property "Footprint" "MagStrike:Gateron_Low_Profile_Magnetic_Jade"
 			(at 93.98 162.56 0)
 			(effects
@@
 			)
 		)
-		(property "Footprint" ""
+		(property "Footprint" "MagStrike:Gateron_Low_Profile_Magnetic_Jade"
 			(at 93.98 189.23 0)
 			(effects
@@
 			)
 		)
-		(property "Footprint" ""
+		(property "Footprint" "MagStrike:Gateron_Low_Profile_Magnetic_Jade"
 			(at 33.02 318.77 0)
 			(effects
@@
 			)
 		)
-		(property "Footprint" ""
+		(property "Footprint" "MagStrike:Gateron_Low_Profile_Magnetic_Jade"
 			(at 33.02 237.49 0)
 			(effects
@@
 			)
 		)
-		(property "Footprint" ""
+		(property "Footprint" "MagStrike:Gateron_Low_Profile_Magnetic_Jade"
 			(at 31.75 341.63 0)
 			(effects
@@
 			)
 		)
-		(property "Footprint" ""
+		(property "Footprint" "MagStrike:Gateron_Low_Profile_Magnetic_Jade"
 			(at 93.98 60.96 0)
 			(effects
@@
 			)
 		)
-		(property "Footprint" ""
+		(property "Footprint" "MagStrike:Gateron_Low_Profile_Magnetic_Jade"
 			(at 124.46 86.36 0)
 			(effects
@@
 			)
 		)
-		(property "Footprint" ""
+		(property "Footprint" "MagStrike:Gateron_Low_Profile_Magnetic_Jade"
 			(at 153.67 138.43 0)
 			(effects
@@
 			)
 		)
-		(property "Footprint" ""
+		(property "Footprint" "MagStrike:Gateron_Low_Profile_Magnetic_Jade"
 			(at 33.02 35.56 0)
 			(effects
@@
 			)
 		)
-		(property "Footprint" ""
+		(property "Footprint" "MagStrike:Gateron_Low_Profile_Magnetic_Jade"
 			(at 63.5 86.36 0)
 			(effects
@@
 			)
 		)
-		(property "Footprint" ""
+		(property "Footprint" "MagStrike:Gateron_Low_Profile_Magnetic_Jade"
 			(at 93.98 86.36 0)
 			(effects
@@
 			)
 		)
-		(property "Footprint" ""
+		(property "Footprint" "MagStrike:Gateron_Low_Profile_Magnetic_Jade"
 			(at 153.67 162.56 0)
 			(effects
@@
 			)
 		)
-		(property "Footprint" ""
+		(property "Footprint" "MagStrike:Gateron_Low_Profile_Magnetic_Jade"
 			(at 93.98 318.77 0)
 			(effects
@@
 			)
 		)
-		(property "Footprint" ""
+		(property "Footprint" "MagStrike:Gateron_Low_Profile_Magnetic_Jade"
 			(at 33.02 111.76 0)
 			(effects
@@
 			)
 		)
-		(property "Footprint" ""
+		(property "Footprint" "MagStrike:Gateron_Low_Profile_Magnetic_Jade"
 			(at 33.02 86.36 0)
 			(effects
@@
 			)
 		)
-		(property "Footprint" ""
+		(property "Footprint" "MagStrike:Gateron_Low_Profile_Magnetic_Jade"
 			(at 124.46 189.23 0)
 			(effects
@@
 			)
 		)
-		(property "Footprint" ""
+		(property "Footprint" "MagStrike:Gateron_Low_Profile_Magnetic_Jade"
 			(at 153.67 86.36 0)
 			(effects
@@
 			)
 		)
-		(property "Footprint" ""
+		(property "Footprint" "MagStrike:Gateron_Low_Profile_Magnetic_Jade"
 			(at 153.67 237.49 0)
 			(effects
@@
 			)
 		)
-		(property "Footprint" ""
+		(property "Footprint" "MagStrike:Gateron_Low_Profile_Magnetic_Jade"
 			(at 153.67 290.83 0)
 			(effects
@@
 			)
 		)
-		(property "Footprint" ""
+		(property "Footprint" "MagStrike:Gateron_Low_Profile_Magnetic_Jade"
 			(at 153.67 213.36 0)
 			(effects
@@
 			)
 		)
-		(property "Footprint" ""
+		(property "Footprint" "MagStrike:Gateron_Low_Profile_Magnetic_Jade"
 			(at 93.98 213.36 0)
 			(effects
@@
 			)
 		)
-		(property "Footprint" ""
+		(property "Footprint" "MagStrike:Gateron_Low_Profile_Magnetic_Jade"
 			(at 93.98 262.89 0)
 			(effects
@@
 			)
 		)
-		(property "Footprint" ""
+		(property "Footprint" "MagStrike:Gateron_Low_Profile_Magnetic_Jade"
 			(at 153.67 111.76 0)
 			(effects
@@
 			)
 		)
-		(property "Footprint" ""
+		(property "Footprint" "MagStrike:Gateron_Low_Profile_Magnetic_Jade"
 			(at 93.98 35.56 0)
 			(effects
@@
 			)
 		)
-		(property "Footprint" ""
+		(property "Footprint" "MagStrike:Gateron_Low_Profile_Magnetic_Jade"
 			(at 33.02 189.23 0)
 			(effects
@@
 			)
 		)
-		(property "Footprint" ""
+		(property "Footprint" "MagStrike:Gateron_Low_Profile_Magnetic_Jade"
 			(at 153.67 35.56 0)
 			(effects
@@
 			)
 		)
-		(property "Footprint" ""
+		(property "Footprint" "MagStrike:Gateron_Low_Profile_Magnetic_Jade"
 			(at 63.5 213.36 0)
 			(effects
@@
 			)
 		)
-		(property "Footprint" ""
+		(property "Footprint" "MagStrike:Gateron_Low_Profile_Magnetic_Jade"
 			(at 93.98 290.83 0)
 			(effects
@@
 			)
 		)
-		(property "Footprint" ""
+		(property "Footprint" "MagStrike:Gateron_Low_Profile_Magnetic_Jade"
 			(at 124.46 318.77 0)
 			(effects
@@
 			)
 		)
-		(property "Footprint" ""
+		(property "Footprint" "MagStrike:Gateron_Low_Profile_Magnetic_Jade"
 			(at 124.46 237.49 0)
 			(effects
@@
 			)
 		)
-		(property "Footprint" ""
+		(property "Footprint" "MagStrike:Gateron_Low_Profile_Magnetic_Jade"
 			(at 63.5 35.56 0)
 			(effects
@@
 			)
 		)
-		(property "Footprint" ""
+		(property "Footprint" "MagStrike:Gateron_Low_Profile_Magnetic_Jade"
 			(at 153.67 60.96 0)
 			(effects
@@
 			)
 		)
-		(property "Footprint" ""
+		(property "Footprint" "MagStrike:Gateron_Low_Profile_Magnetic_Jade"
 			(at 124.46 213.36 0)
 			(effects
@@
 			)
 		)
-		(property "Footprint" ""
+		(property "Footprint" "MagStrike:Gateron_Low_Profile_Magnetic_Jade"
 			(at 63.5 237.49 0)
 			(effects
@@
 			)
 		)
-		(property "Footprint" ""
+		(property "Footprint" "MagStrike:Gateron_Low_Profile_Magnetic_Jade"
 			(at 124.46 138.43 0)
 			(effects
@@
 			)
 		)
-		(property "Footprint" ""
+		(property "Footprint" "MagStrike:Gateron_Low_Profile_Magnetic_Jade"
 			(at 124.46 262.89 0)
 			(effects
@@
 			)
 		)
-		(property "Footprint" ""
+		(property "Footprint" "MagStrike:Gateron_Low_Profile_Magnetic_Jade"
 			(at 63.5 290.83 0)
 			(effects
@@
 			)
 		)
-		(property "Footprint" ""
+		(property "Footprint" "MagStrike:Gateron_Low_Profile_Magnetic_Jade"
 			(at 124.46 111.76 0)
 			(effects
@@
 			)
 		)
-		(property "Footprint" ""
+		(property "Footprint" "MagStrike:Gateron_Low_Profile_Magnetic_Jade"
 			(at 153.67 189.23 0)
 			(effects
@@
 			)
 		)
-		(property "Footprint" ""
+		(property "Footprint" "MagStrike:Gateron_Low_Profile_Magnetic_Jade"
 			(at 63.5 189.23 0)
 			(effects
@@
 			)
 		)
-		(property "Footprint" ""
+		(property "Footprint" "MagStrike:Gateron_Low_Profile_Magnetic_Jade"
 			(at 124.46 162.56 0)
 			(effects
@@
 			)
 		)
-		(property "Footprint" ""
+		(property "Footprint" "MagStrike:Gateron_Low_Profile_Magnetic_Jade"
 			(at 63.5 111.76 0)
 			(effects
@@
 			)
 		)
-		(property "Footprint" ""
+		(property "Footprint" "MagStrike:Gateron_Low_Profile_Magnetic_Jade"
 			(at 93.98 111.76 0)
 			(effects
@@
 			)
 		)
-		(property "Footprint" ""
+		(property "Footprint" "MagStrike:Gateron_Low_Profile_Magnetic_Jade"
 			(at 153.67 318.77 0)
 			(effects
@@
 			)
 		)
-		(property "Footprint" ""
+		(property "Footprint" "MagStrike:Gateron_Low_Profile_Magnetic_Jade"
 			(at 33.02 60.96 0)
 			(effects
@@
 			)
 		)
-		(property "Footprint" ""
+		(property "Footprint" "MagStrike:Gateron_Low_Profile_Magnetic_Jade"
 			(at 93.98 138.43 0)
 			(effects
@@
 			)
 		)
-		(property "Footprint" ""
+		(property "Footprint" "MagStrike:Gateron_Low_Profile_Magnetic_Jade"
 			(at 33.02 213.36 0)
 			(effects
@@
 			)
 		)
-		(property "Footprint" ""
+		(property "Footprint" "MagStrike:Gateron_Low_Profile_Magnetic_Jade"
 			(at 124.46 290.83 0)
 			(effects
@@
 			)
 		)
-		(property "Footprint" ""
+		(property "Footprint" "MagStrike:Gateron_Low_Profile_Magnetic_Jade"
 			(at 93.98 237.49 0)
 			(effects
@@
 			)
 		)
-		(property "Footprint" ""
+		(property "Footprint" "MagStrike:Gateron_Low_Profile_Magnetic_Jade"
 			(at 124.46 35.56 0)
 			(effects

Commit message: some sad things
i have my pcb but relised i have done the pinout wrong
Connections:
- net GND: now also SW1.3 (GND), SW10.3 (GND), SW11.3 (GND), SW12.3 (GND), SW13.3 (GND), SW14.3 (GND), SW15.3 (GND), SW16.3 (GND), SW17.3 (GND), SW18.3 (GND), SW19.3 (GND), SW2.3 (GND), SW20.3 (GND), SW21.3 (GND), SW22.3 (GND), SW23.3 (GND), SW24.3 (GND), SW25.3 (GND), SW26.3 (GND), SW27.3 (GND), SW28.3 (GND), SW29.3 (GND), SW3.3 (GND), SW30.3 (GND), SW31.3 (GND), SW32.3 (GND), SW33.3 (GND), SW34.3 (GND), SW35.3 (GND), SW36.3 (GND), SW37.3 (GND), SW38.3 (GND), SW39.3 (GND), SW4.3 (GND), SW40.3 (GND), SW41.3 (GND), SW42.3 (GND), SW43.3 (GND), SW44.3 (GND), SW45.3 (GND), SW46.3 (GND), SW47.3 (GND), SW48.3 (GND), SW49.3 (GND), SW5.3 (GND), SW50.3 (GND), SW51.3 (GND), SW52.3 (GND), SW53.3 (GND), SW54.3 (GND), SW55.3 (GND), SW56.3 (GND), SW57.3 (GND), SW58.3 (GND), SW59.3 (GND), SW6.3 (GND), SW60.3 (GND), SW61.3 (GND), SW7.3 (GND), SW8.3 (GND), SW9.3 (GND); no longer SW1.2 (GND), SW10.2 (GND), SW11.2 (GND), SW12.2 (GND), SW13.2 (GND), SW14.2 (GND), SW15.2 (GND), SW16.2 (GND), SW17.2 (GND), SW18.2 (GND), SW19.2 (GND), SW2.2 (GND), SW20.2 (GND), SW21.2 (GND), SW22.2 (GND), SW23.2 (GND), SW24.2 (GND), SW25.2 (GND), SW26.2 (GND), SW27.2 (GND), SW28.2 (GND), SW29.2 (GND), SW3.2 (GND), SW30.2 (GND), SW31.2 (GND), SW32.2 (GND), SW33.2 (GND), SW34.2 (GND), SW35.2 (GND), SW36.2 (GND), SW37.2 (GND), SW38.2 (GND), SW39.2 (GND), SW4.2 (GND), SW40.2 (GND), SW41.2 (GND), SW42.2 (GND), SW43.2 (GND), SW44.2 (GND), SW45.2 (GND), SW46.2 (GND), SW47.2 (GND), SW48.2 (GND), SW49.2 (GND), SW5.2 (GND), SW50.2 (GND), SW51.2 (GND), SW52.2 (GND), SW53.2 (GND), SW54.2 (GND), SW55.2 (GND), SW56.2 (GND), SW57.2 (GND), SW58.2 (GND), SW59.2 (GND), SW6.2 (GND), SW60.2 (GND), SW61.2 (GND), SW7.2 (GND), SW8.2 (GND), SW9.2 (GND)
- net SW1: now also SW1.2 (OUT); no longer SW1.3 (OUT)
- net SW10: now also SW10.2 (OUT); no longer SW10.3 (OUT)
- net SW11: now also SW11.2 (OUT); no longer SW11.3 (OUT)
- net SW12: now also SW12.2 (OUT); no longer SW12.3 (OUT)
- net SW13: now also SW13.2 (OUT); no longer SW13.3 (OUT)
- net SW14: now also SW14.2 (OUT); no longer SW14.3 (OUT)
- net SW15: no longer SW15.3 (OUT)
- net SW16: now also SW16.2 (OUT); no longer SW16.3 (OUT)
- net SW17: now also SW17.2 (OUT); no longer SW17.3 (OUT)
- net SW18: now also SW18.2 (OUT); no longer SW18.3 (OUT)
- net SW19: now also SW19.2 (OUT); no longer SW19.3 (OUT)
- net SW2: now also SW2.2 (OUT); no longer SW2.3 (OUT)
- net SW20: now also SW20.2 (OUT); no longer SW20.3 (OUT)
- net SW21: now also SW21.2 (OUT); no longer SW21.3 (OUT)
- net SW22: now also SW22.2 (OUT); no longer SW22.3 (OUT)
- net SW23: now also SW23.2 (OUT); no longer SW23.3 (OUT)
- net SW24: now also SW24.2 (OUT); no longer SW24.3 (OUT)
- net SW25: now also SW25.2 (OUT); no longer SW25.3 (OUT)
- net SW26: now also SW26.2 (OUT); no longer SW26.3 (OUT)
- net SW27: now also SW27.2 (OUT); no longer SW27.3 (OUT)
- net SW28: now also SW28.2 (OUT); no longer SW28.3 (OUT)
- net SW29: now also SW29.2 (OUT); no longer SW29.3 (OUT)
- net SW3: now also SW3.2 (OUT); no longer SW3.3 (OUT)
- net SW30: now also SW30.2 (OUT); no longer SW30.3 (OUT)
- net SW31: now also SW31.2 (OUT); no longer SW31.3 (OUT)
- net SW32: now also SW32.2 (OUT); no longer SW32.3 (OUT)
- net SW33: now also SW33.2 (OUT); no longer SW33.3 (OUT)
- net SW34: now also SW34.2 (OUT); no longer SW34.3 (OUT)
- net SW35: now also SW35.2 (OUT); no longer SW35.3 (OUT)
- net SW36: now also SW36.2 (OUT); no longer SW36.3 (OUT)
- net SW37: now also SW37.2 (OUT); no longer SW37.3 (OUT)
- net SW38: now also SW38.2 (OUT); no longer SW38.3 (OUT)
- net SW39: now also SW39.2 (OUT); no longer SW39.3 (OUT)
- net SW4: now also SW4.2 (OUT); no longer SW4.3 (OUT)
- net SW40: now also SW40.2 (OUT); no longer SW40.3 (OUT)
- net SW41: now also SW41.2 (OUT); no longer SW41.3 (OUT)
- net SW42: now also SW42.2 (OUT); no longer SW42.3 (OUT)
- net SW43: now also SW43.2 (OUT); no longer SW43.3 (OUT)
- net SW44: now also SW44.2 (OUT); no longer SW44.3 (OUT)
- net SW45: now also SW45.2 (OUT); no longer SW45.3 (OUT)
- net SW46: now also SW46.2 (OUT); no longer SW46.3 (OUT)
- net SW47: now also SW47.2 (OUT); no longer SW47.3 (OUT)
- net SW48: now also SW48.2 (OUT); no longer SW48.3 (OUT)
- net SW49: now also SW49.2 (OUT); no longer SW49.3 (OUT)
- net SW5: now also SW15.2 (OUT), SW5.2 (OUT); no longer SW5.3 (OUT)
- net SW50: now also SW50.2 (OUT); no longer SW50.3 (OUT)
- net SW51: now also SW51.2 (OUT); no longer SW51.3 (OUT)
- net SW52: now also SW52.2 (OUT); no longer SW52.3 (OUT)
- net SW53: now also SW53.2 (OUT); no longer SW53.3 (OUT)
- net SW54: now also SW54.2 (OUT); no longer SW54.3 (OUT)
- net SW55: now also SW55.2 (OUT); no longer SW55.3 (OUT)
- net SW56: now also SW56.2 (OUT); no longer SW56.3 (OUT)
- net SW57: now also SW57.2 (OUT); no longer SW57.3 (OUT)
- net SW58: now also SW58.2 (OUT); no longer SW58.3 (OUT)
- net SW59: now also SW59.2 (OUT); no longer SW59.3 (OUT)
- net SW6: now also SW6.2 (OUT); no longer SW6.3 (OUT)
- net SW60: now also SW60.2 (OUT); no longer SW60.3 (OUT)
- net SW61: now also SW61.2 (OUT); no longer SW61.3 (OUT)
- net SW7: now also SW7.2 (OUT); no longer SW7.3 (OUT)
- net SW8: now also SW8.2 (OUT); no longer SW8.3 (OUT)
- net SW9: now also SW9.2 (OUT); no longer SW9.3 (OUT)
Other:
- moved on the sheet: SW1

Commit message: more stuff
mores stutff
Connections:
- net SW15: now also SW15.2 (OUT)
- net SW5: no longer SW15.2 (OUT)
Changed lines of the file:
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@@
 		)
 	)
-	(global_label "SW5"
+	(global_label "SW15"
 		(shape input)
 		(at 191.77 245.11 180)
@@
 		)
 		(property "Intersheetrefs" "${INTERSHEET_REFS}"
-			(at 184.9144 245.11 0)
+			(at 183.7049 245.11 0)
 			(effects
 				(font
