File: PCB/MagStrike.kicad_pcb (KiCad board)
At the start: 2 copper layers, 485.8 x 326.2 mm, 67 parts, among them U1 CD74HC4067M, U2 CD74HC4067M, U3 CD74HC4067M, U4 CD74HC4067M

Commit message: and
Parts:
- removed REF**: 2U, Stablilizer:2U
- A1: moved to F.Cu
- U1, U2, U3, U4: moved to B.Cu
- moved A1 223.5 mm to (56.5, 17.6), turned to 90 degrees
- moved U1 134.7 mm to (138.8, 85.5), turned to -90 degrees
- moved U4 129.8 mm to (203.6, 85.3), turned to -90 degrees
- moved U3 83.6 mm to (180.7, 85.3), turned to -90 degrees
- moved U2 51.4 mm to (159.5, 85.4), turned to -90 degrees
Routing:
- net GND: track 0.00 -> 294.5 mm, vias 0 -> 11
- net +3V3: track 0.00 -> 282.7 mm
- net SW14: track 0.00 -> 248.4 mm, vias 0 -> 1
- net SW13: track 0.00 -> 217.6 mm, vias 0 -> 3
- net SW12: track 0.00 -> 202.7 mm, vias 0 -> 1
- net SW11: track 0.00 -> 184.6 mm, vias 0 -> 1
- net SW6: track 0.00 -> 158.8 mm, vias 0 -> 1
- net SW5: track 0.00 -> 137.1 mm, vias 0 -> 1
- net SW10: track 0.00 -> 133.9 mm, vias 0 -> 1
- net SW2: track 0.00 -> 124.5 mm, vias 0 -> 1
- net SW9: track 0.00 -> 123.2 mm, vias 0 -> 1
- net SW1: track 0.00 -> 119.7 mm, vias 0 -> 1
- net SW4: track 0.00 -> 111.7 mm, vias 0 -> 1
- net SW8: track 0.00 -> 95.0 mm, vias 0 -> 1
- net SW3: track 0.00 -> 94.9 mm, vias 0 -> 1
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Other:
- board size 485.8 x 326.2 mm -> 667.9 x 227.8 mm

Commit message: df
Routing:
- net +3V3: track 282.7 -> 1515.7 mm, vias 0 -> 24
- net GND: track 294.5 -> 1482.6 mm, vias 11 -> 30
- net SW54: track 0.00 -> 189.9 mm, vias 0 -> 1
- net GPIO15: track 0.00 -> 183.3 mm, vias 0 -> 3
- net SW28: track 0.00 -> 177.2 mm, vias 0 -> 1
- net GPI014: track 0.00 -> 172.0 mm, vias 0 -> 1
- net SW42: track 0.00 -> 162.6 mm, vias 0 -> 1
- net SW55: track 0.00 -> 162.0 mm, vias 0 -> 1
- net SW27: track 0.00 -> 153.1 mm, vias 0 -> 1
- net SW29: track 0.00 -> 142.2 mm, vias 0 -> 1
- net SW56: track 0.00 -> 142.1 mm, vias 0 -> 1
- net SW41: track 0.00 -> 133.1 mm, vias 0 -> 1
- net SW26: track 0.00 -> 132.3 mm, vias 0 -> 1
- net SW43: track 0.00 -> 132.1 mm, vias 0 -> 1
- net SW61: track 0.00 -> 124.7 mm, vias 0 -> 1
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
Commit message: ds
Routing:
- net GPI09: track 0.00 -> 249.5 mm, vias 0 -> 12
- net GPI011: track 0.00 -> 238.5 mm, vias 0 -> 7
- net GPI08: track 0.00 -> 233.3 mm, vias 0 -> 13
- net GPI010: track 0.00 -> 215.7 mm, vias 0 -> 11
- net GPI013: track 0.00 -> 147.4 mm, vias 0 -> 7
- net GPI012: track 0.00 -> 121.7 mm, vias 0 -> 5
- net GPI026: track 0.00 -> 118.8 mm, vias 0 -> 14
- net SW57: track 0.00 -> 72.4 mm, vias 0 -> 1
- net +3V3: track 1515.7 -> 1522.7 mm
- net GND: track 1482.6 -> 1487.4 mm, vias 30 -> 32
- net SW19: track 63.7 -> 65.3 mm
- net SW11: track 184.6 -> 185.7 mm
- net SW34: track 40.6 -> 39.6 mm

Commit message: a
Other:
- board size 667.9 x 227.8 mm -> 285.8 x 119.8 mm
Changed lines of the file:
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@@
 		)
 	)
-	(gr_rect
-		(start -147.3325 -38.12)
-		(end 520.519316 189.67)
+	(gr_line
+		(start 27.98 5.786102)
+		(end 27.98 123.358092)
 		(stroke
 			(width 0.05)
 			(type default)
 		)
-		(fill no)
 		(layer "Edge.Cuts")
 	)
+	(gr_arc
+		(start 29.116102 124.403898)
+		(mid 28.31 124.07)
+		(end 27.976102 123.263898)
+		(stroke
+			(width 0.05)
+			(type default)
+		)
+		(layer "Edge.Cuts")
+	)
+	(gr_arc
+		(start 85.916102 27.823898)
+		(mid 85.11 27.49)
+		(end 84.776102 26.683898)
+		(stroke
+			(width 0.05)
+			(type default)
+		)
+		(layer "Edge.Cuts")
+	)
+	(gr_line
+		(start 313.749566 123.363192)
+		(end 313.71 28.84)
+		(stroke
+			(width 0.05)
+			(type default)
+		)
+		(layer "Edge.Cuts")
+	)
+	(gr_arc
+		(start 83.623898 4.676102)
+		(mid 84.43 5.01)
+		(end 84.763898 5.816102)
+		(stroke
+			(width 0.05)
+			(type default)
+		)
+		(layer "Edge.Cuts")
+	)
+	(gr_line
+		(start 29.021908 124.4)
+		(end 312.708092 124.4)
+		(stroke
+			(width 0.05)
+			(type default)
+		)
+		(layer "Edge.Cuts")
+	)
+	(gr_arc
+		(start 313.753898 123.263898)
+		(mid 313.42 124.07)
+		(end 312.613898 124.403898)
+		(stroke
+			(width 0.05)
+			(type default)
+		)
+		(layer "Edge.Cuts")
+	)
+	(gr_line
+		(start 84.776103 26.683898)
+		(end 84.77 4.68)
+		(stroke
+			(width 0.05)
+			(type default)
+		)
+		(layer "Edge.Cuts")
+	)
+	(gr_line
+		(start 312.57 27.7)
+		(end 85.916102 27.819396)
+		(stroke
+			(width 0.05)
+			(type default)
+		)
+		(layer "Edge.Cuts")
+	)
+	(gr_arc
+		(start 312.57 27.7)
+		(mid 313.376102 28.033898)
+		(end 313.71 28.84)
+		(stroke
+			(width 0.05)
+			(type default)
+		)
+		(layer "Edge.Cuts")
+	)
+	(gr_line
+		(start 83.623898 4.676102)
+		(end 28.956788 4.660344)
+		(stroke
+			(width 0.05)
+			(type default)
+		)
+		(layer "Edge.Cuts")
+	)
+	(gr_arc
+		(start 27.996102 5.786102)
+		(mid 28.33 4.98)
+		(end 29.136102 4.646102)
+		(stroke
+			(width 0.05)
+			(type default)
+		)
+		(layer "Edge.Cuts")
+	)

Commit message: a
Parts:
- added REF**: 2U, Stablilizer:2U, F.Cu at (294.4, 76.0)
- added REF**: 2U, Stablilizer:2U, F.Cu at (296.8, 37.9)
- added REF**: 6U, Stablilizer:6U, F.Cu at (162.7, 99.2)
- added REF**: 2U, Stablilizer:2U, F.Cu at (51.4, 95.1)
- added REF**: 2U, Stablilizer:2U, F.Cu at (289.6, 95.1)
Routing:
- net GND: track 1487.4 -> 1517.5 mm, vias 32 -> 34
- net +3V3: track 1522.7 -> 1550.2 mm
- net SW58: track 79.1 -> 95.1 mm
- net SW56: track 142.1 -> 146.7 mm
- net SW53: track 97.4 -> 100.9 mm
- net SW60: track 109.0 -> 112.2 mm
- net SW41: track 133.1 -> 135.5 mm
- net SW14: track 248.6 -> 250.5 mm
- net GPI09: track 249.5 -> 250.8 mm, vias 12 -> 14
- net GPIO15: track 183.3 -> 184.3 mm
Other:
- board size 285.8 x 119.8 mm -> 288.7 x 121.5 mm
