File: PCB/MagStrike.kicad_pcb (KiCad board)
At the start: 2 copper layers, 288.7 x 121.5 mm, 67 parts, among them U1 CD74HC4067M, U2 CD74HC4067M, U3 CD74HC4067M, U4 CD74HC4067M

Commit message: S
Routing:
- net +3V3: track 0.00 -> 489.8 mm, vias 0 -> 6
- net GND: track 0.00 -> 464.9 mm, vias 0 -> 27
- net SW14: track 0.00 -> 296.9 mm, vias 0 -> 2
- net SW13: track 0.00 -> 268.9 mm, vias 0 -> 2
- net SW12: track 0.00 -> 250.0 mm
- net SW11: track 0.00 -> 240.1 mm
- net SW10: track 0.00 -> 235.7 mm
- net SW9: track 0.00 -> 224.8 mm
- net SW8: track 0.00 -> 204.9 mm
- net SW7: track 0.00 -> 185.3 mm
- net SW6: track 0.00 -> 170.1 mm
- net SW21: track 0.00 -> 160.2 mm, vias 0 -> 2
- net SW1: track 0.00 -> 154.8 mm
- net SW20: track 0.00 -> 142.8 mm, vias 0 -> 2
- net SW5: track 0.00 -> 141.3 mm, vias 0 -> 2
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Other:
- board text added: "SW10"
- board text added: "SW11"
- board text added: "SW12"
- board text added: "SW13"
- board text added: "SW14"
- board text added: "SW2"
- board text added: "SW3"
- board text added: "SW4"
- board text added: "SW5"
- board text added: "SW6"
- board text added: "SW7"
- board text added: "SW8"
- board text added: "SW9"
- board text removed: "${REFERENCE}"

Commit message: alnm sdklnsdjklsdf
more traces 👍
Routing:
- net +3V3: track 489.8 -> 1290.0 mm, vias 6 -> 25
- net GND: track 464.9 -> 1212.7 mm, vias 27 -> 86
- net SW28: track 0.00 -> 289.9 mm, vias 0 -> 2
- net SW27: track 0.00 -> 271.1 mm, vias 0 -> 2
- net SW41: track 0.00 -> 261.4 mm, vias 0 -> 2
- net SW26: track 0.00 -> 256.0 mm, vias 0 -> 2
- net SW25: track 0.00 -> 241.0 mm, vias 0 -> 4
- net SW24: track 0.00 -> 218.8 mm, vias 0 -> 2
- net SW40: track 0.00 -> 215.9 mm, vias 0 -> 1
- net SW39: track 0.00 -> 199.8 mm, vias 0 -> 2
- net SW23: track 0.00 -> 198.4 mm, vias 0 -> 2
- net SW42: track 0.00 -> 184.9 mm, vias 0 -> 1
- net SW38: track 0.00 -> 180.2 mm, vias 0 -> 2
- net SW22: track 0.00 -> 179.7 mm, vias 0 -> 2
- net SW37: track 0.00 -> 157.0 mm, vias 0 -> 2
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
Commit message: more traces
more traces
Routing:
- net +3V3: track 1290.0 -> 1545.3 mm, vias 25 -> 33
- net GND: track 1212.7 -> 1463.0 mm, vias 86 -> 100
- net GPI012: track 0.00 -> 157.6 mm, vias 0 -> 3
- net SW61: track 0.00 -> 147.8 mm, vias 0 -> 4
- net SW60: track 0.00 -> 141.6 mm, vias 0 -> 3
- net SW55: track 0.00 -> 127.1 mm, vias 0 -> 2
- net SW59: track 0.00 -> 111.1 mm, vias 0 -> 3
- net SW56: track 0.00 -> 104.0 mm, vias 0 -> 2
- net GPI026: track 0.00 -> 98.8 mm, vias 0 -> 8
- net GPI08: track 0.00 -> 94.5 mm, vias 0 -> 6
- net GPI09: track 0.00 -> 94.2 mm, vias 0 -> 9
- net GPI010: track 0.00 -> 92.2 mm, vias 0 -> 8
- net GPI011: track 0.00 -> 87.3 mm, vias 0 -> 5
- net SW58: track 0.00 -> 68.6 mm, vias 0 -> 3
- net SW57: track 0.00 -> 28.9 mm, vias 0 -> 2
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